File: PCBs/Sedna Power Board.sch (EAGLE design)
At the start: 21 parts

Commit message: Finished the 12v and 7.2v circuits, started working on the current sensing setup
Parts:
- added CURRENT_GAUGE: CS70, Sedna Components:CS70
- added C_OUT_12, C_OUT_5_A, C_OUT_5_B, C_OUT_7.2_A: 47μF, 16V, Sedna Components:GRM32
- added C_OUT_7.2_B: 22μF, 16V, Sedna Components:GRM31
- added R_FBH_12: 619kΩ, 0.1%, rcl:R-US_R0805
- added R_FBH_7.2: 680kΩ, 0.1%, rcl:R-US_R0805
- added R_FBL_12: 47kΩ, 0.1%, rcl:R-US_R0805
- added R_FBL_7.2: 91kΩ, 0.1%, rcl:R-US_R0805
- added R_PGOOD_12, R_PGOOD_5, R_PGOOD_7.2: 1MΩ, 1%, rcl:R-US_R0805
- added R_SENSE: 12mΩ, 1%, 300mW, Sedna Components:WSK1206
Connections:
- removed net VIN: C_PF1.2, L_PF1.1
- new net +10V: 12V_REGULATOR.VBIAS, 7.2V_REGULATOR.VBIAS, CURRENT_GAUGE.SEL1, CURRENT_GAUGE.VCC+, C_OUT_12.1, C_OUT_7.2_A.1, C_OUT_7.2_B.1, C_PF1.2, L_12.2, L_7.2.2, L_PF1.1, R_FBH_12.2, R_FBH_7.2.2, R_PGOOD_12.2, R_PGOOD_7.2.2
- new net N$14: 7.2V_REGULATOR.PGOOD, R_PGOOD_7.2.1
- new net N$15: 5V_REGULATOR.PGOOD, R_PGOOD_5.1
- new net N$17: 12V_REGULATOR.VOUT/FB, R_FBH_12.1, R_FBL_12.2
- new net N$19: 7.2V_REGULATOR.VOUT/FB, R_FBH_7.2.1, R_FBL_7.2.2
- new net N$20: CURRENT_GAUGE.VP, C_IN.2, C_PF3.2, C_PF4.+, L_PF2.2, R_SENSE.1
- new net N$21: CURRENT_GAUGE.OUT
- new net N$5: 12V_REGULATOR.PGOOD, R_PGOOD_12.1
- net GND: now also CURRENT_GAUGE.GND, CURRENT_GAUGE.SEL2, CURRENT_GAUGE.VCC-, C_OUT_12.2, C_OUT_7.2_A.2, C_OUT_7.2_B.2, R_FBL_12.1, R_FBL_7.2.1
- net N$13: now also CURRENT_GAUGE.VM, R_SENSE.2; no longer C_IN.2, C_PF3.2, C_PF4.+, L_PF2.2

Commit message: I decided the giant monolithic PCB isn't the way to start, so I started making individual breakout-style boards for all of the SMDs. Meet v1.0 of the L6983 power board!
Parts:
- added TEMP_SENSOR: TC77, Sedna Components:TC77
Changed lines of the file:
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@@
 <layer number="112" name="tSilk" color="7" fill="1" visible="yes" active="yes"/>
 <layer number="113" name="IDFDebug" color="4" fill="1" visible="yes" active="yes"/>
+<layer number="114" name="Badge_Outline" color="7" fill="1" visible="yes" active="yes"/>
+<layer number="115" name="ReferenceISLANDS" color="7" fill="1" visible="yes" active="yes"/>
 <layer number="116" name="Patch_BOT" color="9" fill="4" visible="yes" active="yes"/>
+<layer number="118" name="Rect_Pads" color="7" fill="1" visible="yes" active="yes"/>
 <layer number="121" name="_tsilk" color="7" fill="1" visible="yes" active="yes"/>
 <layer number="122" name="_bsilk" color="7" fill="1" visible="yes" active="yes"/>
@@
 <part name="SUPPLY2" library="Sedna Components" deviceset="VIN/VOUT_2" device="" value="+3.3V IN"/>
 <part name="GND9" library="supply1" library_urn="urn:adsk.eagle:library:371" deviceset="GND" device=""/>
+<part name="TEMP_SENSOR" library="Sedna Components" deviceset="TC77" device=""/>
 </parts>
 <sheets>
@@
 <attribute name="VALUE" x="7.62" y="40.64" size="1.778" layer="96"/>
 </instance>
+<instance part="TEMP_SENSOR" gate="G$1" x="30.48" y="17.78" smashed="yes">
+<attribute name="NAME" x="20.32" y="23.876" size="1.778" layer="95"/>
+<attribute name="VALUE" x="20.32" y="7.62" size="1.778" layer="96"/>
+</instance>
 </instances>
