File: PCBs/L6983 Regulator Board.sch (EAGLE design)
At the start: 23 parts

Commit message: Now that the laser engraver is done, I can start fabricating some boards. Updated the power board to v1.1, put together a BOM to make 3 of them at 12v, 7.2v, and 5v.
Parts:
- C_IN: device rcl:C-EUC0805 -> rcl:C-EUC1206
Changed lines of the file:
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@@
 <?xml version="1.0" encoding="utf-8"?>
 <!DOCTYPE eagle SYSTEM "eagle.dtd">
-<eagle version="9.6.0">
+<eagle version="9.6.1">
 <drawing>
 <settings>
@@
 <part name="R_FILT" library="rcl" library_urn="urn:adsk.eagle:library:334" deviceset="R-US_" device="R0805" package3d_urn="urn:adsk.eagle:package:23553/2" value="100Ω"/>
 <part name="C_FILT" library="rcl" library_urn="urn:adsk.eagle:library:334" deviceset="C-EU" device="C0805" package3d_urn="urn:adsk.eagle:package:23617/2" value="1μF, 50v"/>
-<part name="C_IN" library="rcl" library_urn="urn:adsk.eagle:library:334" deviceset="C-EU" device="C0805" package3d_urn="urn:adsk.eagle:package:23617/2" value="10μF, 50v"/>
+<part name="C_IN" library="rcl" library_urn="urn:adsk.eagle:library:334" deviceset="C-EU" device="C1206" package3d_urn="urn:adsk.eagle:package:23618/2" value="10μF, 50v"/>
 <part name="C_BOOT" library="rcl" library_urn="urn:adsk.eagle:library:334" deviceset="C-EU" device="C0805" package3d_urn="urn:adsk.eagle:package:23617/2" value="100nF, 50v"/>
 <part name="L_OUT" library="Sedna Components" deviceset="PA4343_FP2" device=""/>
